File: sw/sm/StationModule.sch (EAGLE design)
At the start: 18 parts, among them CN1 USB-Pigtail connection, IC1 REG1117

Commit message: Updated SM
Parts:
- added JP3: (no value), pinhead:PINHD-1X3
- added R5, R7: 10k, rcl:R-US_R0805
- added R6: 1k, rcl:R-US_R0805
- added T1: 2N3904, transistor:2N3904
Connections:
- new net APD-ENABLE: R5.1, T1.C
- new net N$1: R5.2
- new net N$2: R6.1, R7.2, T1.B
- net GND: now also JP3.3, R7.1, T1.E
Other:
- note added: "APD Interface"
- moved on the sheet: JP1, JP2, JP6

Commit message: SM rev1
Parts:
- removed CN1: USB-Pigtail connection, adafruit:1X4-3.5MM
- removed CN2: (no value), adafruit:DCBARRELPTH
- removed D1: (no value), adafruit:DIODESOT23_WAVE
- removed D2: DZ2405100LCT-ZENER, _VMS:DZ2405100LCT-ZENER
- removed JP1, JP2, JP6: (no value), pinhead+:PINHD-1X51X05_SMT
- removed R5, R7: 10k, rcl:R-US_R0805
- removed R6: 1k, rcl:R-US_R0805
- removed T1: 2N3904, transistor:2N3904
- added C4, C5: 100n, rcl:C-EUC0805K
- added H1, H2, H3, H4: MOUNT-HOLE3.0, holes:MOUNT-HOLE3.0
- added PROG-HEADER: PROG-HEADER, pinhead+:PINHD-1X6
- added RFID-HEADER: RFID-HEADER, pinhead+:PINHD-1X6
- added SPI-HEADER: SPI_HEADER, pinhead+:PINHD-1X5
- added SPI_HEADER: SPI-HEADER, pinhead+:PINHD-1X5
- added U$1, U$2: 4050B, Ty2017:4050B
- added USB: USB-HEADER, pinhead+:PINHD-1X4
- JP3: value (none) -> APD-HEADER
- R2, R3: value (none) -> 10k
Connections:
- removed net +12V: CN2.PWR, D1.A, D1.C, D2.A, D2.C
- removed net APD-ENABLE: R5.1, T1.C
- removed net ESPFLASH: JP6.5, R1.1, S2.1, U1.GPIO0
- removed net ESPRESET: JP6.4, R4.1, S1.2, U1.RESET
- removed net N$1: R5.2
- removed net N$12: U1.GPIO13
- removed net N$13: U1.GPIO12
- removed net N$14: U1.ADC
- removed net N$15: U1.GPIO14
- removed net N$16: U1.GPIO16
- removed net N$2: R6.1, R7.2, T1.B
- removed net N$3: R2.1, U1.GPIO15
- removed net N$9: R3.1, U1.GPIO2
- removed net RX: JP6.2, U1.RX
- removed net TX: JP6.1, U1.TX
- removed net V+: JP1.1
- new net APD_EN: JP3.1, U$2G$1.P$2
- new net BUZZER: RFID-HEADER.4, U$2G$3.P$2
- new net GPIO0: PROG-HEADER.1, R1.1, S2.1, U$2G$2.P$1, U1.GPIO0
- new net GPIO1: PROG-HEADER.3, SPI-HEADER.4, SPI_HEADER.4, U1.TX
- new net GPIO12: SPI-HEADER.2, SPI_HEADER.2, U1.GPIO12
- new net GPIO13: SPI-HEADER.3, SPI_HEADER.3, U1.GPIO13
- new net GPIO14: SPI-HEADER.1, SPI_HEADER.1, U1.GPIO14
- new net GPIO15: R2.1, U$2G$1.P$1, U1.GPIO15
- new net GPIO2: R3.1, U$2G$3.P$1, U1.GPIO2
- new net GPIO3: PROG-HEADER.5, SPI-HEADER.5, SPI_HEADER.5, U1.RX
- new net GREEN_LED: RFID-HEADER.5, U$2G$2.P$2
- new net RESET: PROG-HEADER.4, R4.1, S1.2, U1.RESET
- net +3V3: now also C4.1, PROG-HEADER.2, U$1G$7.PWR
- net +5V: now also C5.1, RFID-HEADER.1, U$2G$7.PWR, USB.1; no longer CN1.1
- net D+: now also USB.2; no longer CN1.2
- net D-: now also USB.3; no longer CN1.3
- net GND: now also C4.2, C5.2, PROG-HEADER.6, RFID-HEADER.6, U$1G$3.P$1, U$1G$4.P$1, U$1G$5.P$1, U$1G$6.P$1, U$1G$7.GND, U$2G$4.P$1, U$2G$5.P$1, U$2G$6.P$1, U$2G$7.GND, U1.ADC, USB.4; no longer CN1.4, JP1.2, JP6.3, R7.1, T1.E
- net GPIO4: now also U$1G$1.P$2
- net GPIO5: now also U$1G$2.P$2
- net RFID-DATA0: now also RFID-HEADER.2, U$1G$2.P$1; no longer JP1.4
- net RFID-DATA1: now also RFID-HEADER.3, U$1G$1.P$1; no longer JP1.3
Other:
- note added: "3.3V to 5V level shifter"
- note added: "5V to 3.3V level shifter"
- note added: "Device power and USB HID"
- note added: "MISO"
- note added: "MOSI"
- note added: "NC"
- note added: "NO CONNECT"
- note added: "SCK"
- note added: "SPI HEADER"
- note added: "SS1"
- note added: "SS2"
- note added: "USB data lines for future peripherals"
- note added: "Unused inputs must be pulled HIGH or LOW"
- note removed: "***ADD PROTECTION***"
- note removed: "Device power and HID"
- note removed: "Optional 12V power supply"
- note removed: "RED-LED GREEN-LED BEEP"
- moved on the sheet: C1, JP3, R1, R2, R3, R4, S1, S2, U1
