File: SM/StationModule.sch (EAGLE design)
At the start: 25 parts, among them IC1 REG1117

Commit message: silkscreen
Parts:
- added D2: PMLL4150, diode:PMLL4150
- added R5: 10k, rcl:R-US_R0805
- added R6: 33k, rcl:R-US_R0805
- added STOP: (no value), pinhead+:PINHD-1X2
Connections:
- new net ADC: D2.A, R5.2, R6.1, U1.ADC
- new net STOP: R6.2, STOP.2
- net +3V3: now also STOP.1
- net GND: now also D2.C, R5.1; no longer U1.ADC
Changed lines of the file:
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@@
 <part name="SUPPLY14" library="supply2" deviceset="GND" device=""/>
 <part name="SUPPLY15" library="supply2" deviceset="GND" device=""/>
-<part name="SUPPLY16" library="supply2" deviceset="GND" device=""/>
 <part name="SPI_HEADER" library="pinhead+" deviceset="PINHD-1X5" device="" value="SPI-HEADER"/>
 <part name="SPI-HEADER" library="pinhead+" deviceset="PINHD-1X5" device="" value="SPI_HEADER"/>
@@
 <part name="H4" library="holes" deviceset="MOUNT-HOLE" device="3.0"/>
 <part name="USB" library="pinhead+" deviceset="PINHD-1X4" device="" value="USB-HEADER"/>
+<part name="STOP" library="pinhead+" deviceset="PINHD-1X2" device=""/>
+<part name="R5" library="rcl" deviceset="R-US_" device="R0805" value="10k"/>
+<part name="R6" library="rcl" deviceset="R-US_" device="R0805" value="33k"/>
+<part name="SUPPLY16" library="supply2" deviceset="GND" device=""/>
+<part name="SUPPLY18" library="supply2" deviceset="GND" device=""/>
+<part name="+3V9" library="supply1" deviceset="+3V3" device=""/>
+<part name="D2" library="diode" deviceset="PMLL4150" device=""/>
 </parts>
 <sheets>
@@
 <instance part="+3V3" gate="G$1" x="86.36" y="38.1"/>
 <instance part="+3V4" gate="G$1" x="121.92" y="35.56"/>
-<instance part="+3V5" gate="G$1" x="20.32" y="30.48"/>
+<instance part="+3V5" gate="G$1" x="20.32" y="35.56"/>
 <instance part="+3V6" gate="G$1" x="22.86" y="12.7" rot="R90"/>
 <instance part="SUPPLY4" gate="GND" x="-116.84" y="99.06"/>
@@
 <instance part="SUPPLY14" gate="GND" x="-38.1" y="86.36"/>
 <instance part="SUPPLY15" gate="GND" x="35.56" y="83.82"/>
-<instance part="SUPPLY16" gate="GND" x="27.94" y="27.94" rot="R270"/>
 <instance part="SPI_HEADER" gate="A" x="-111.76" y="-33.02"/>
 <instance part="SPI-HEADER" gate="A" x="-91.44" y="-33.02"/>
@@
 <instance part="H4" gate="G$1" x="119.38" y="-93.98"/>
 <instance part="USB" gate="A" x="-106.68" y="106.68"/>
+<instance part="STOP" gate="G$1" x="-50.8" y="27.94"/>
+<instance part="R5" gate="G$1" x="5.08" y="22.86" rot="R90"/>
+<instance part="R6" gate="G$1" x="-15.24" y="27.94" rot="R180"/>
+<instance part="SUPPLY16" gate="GND" x="-7.62" y="15.24"/>
+<instance part="SUPPLY18" gate="GND" x="5.08" y="15.24"/>
+<instance part="+3V9" gate="G$1" x="-40.64" y="38.1"/>
+<instance part="D2" gate="G$1" x="-7.62" y="22.86" rot="R270"/>
 </instances>
 <busses>
@@
 </segment>
 <segment>
-<pinref part="U1" gate="G$1" pin="ADC"/>
-<wire x1="35.56" y1="27.94" x2="30.48" y2="27.94" width="0.1524" layer="91"/>
-<pinref part="SUPPLY16" gate="GND" pin="GND"/>
-</segment>
-<segment>
 <pinref part="PROG-HEADER" gate="A" pin="6"/>
 <pinref part="SUPPLY17" gate="GND" pin="GND"/>
 <wire x1="-99.06" y1="63.5" x2="-121.92" y2="63.5" width="0.1524" layer="91"/>
+</segment>
+<segment>
+<pinref part="R5" gate="G$1" pin="1"/>
+<pinref part="SUPPLY18" gate="GND" pin="GND"/>
+</segment>
+<segment>
+<pinref part="SUPPLY16" gate="GND" pin="GND"/>
+<pinref part="D2" gate="G$1" pin="C"/>
+<wire x1="-7.62" y1="20.32" x2="-7.62" y2="17.78" width="0.1524" layer="91"/>
 </segment>
 </net>
@@
 <pinref part="U1" gate="G$1" pin="CH_PD"/>
 <wire x1="35.56" y1="25.4" x2="20.32" y2="25.4" width="0.1524" layer="91"/>
-<wire x1="20.32" y1="25.4" x2="20.32" y2="27.94" width="0.1524" layer="91"/>
+<wire x1="20.32" y1="25.4" x2="20.32" y2="33.02" width="0.1524" layer="91"/>
 <pinref part="+3V5" gate="G$1" pin="+3V3"/>
 </segment>
@@
 <wire x1="-99.06" y1="73.66" x2="-121.92" y2="73.66" width="0.1524" layer="91"/>
 </segment>
+<segment>
+<pinref part="STOP" gate="G$1" pin="1"/>
+<wire x1="-53.34" y1="30.48" x2="-40.64" y2="30.48" width="0.1524" layer="91"/>
+<pinref part="+3V9" gate="G$1" pin="+3V3"/>
+<wire x1="-40.64" y1="35.56" x2="-40.64" y2="30.48" width="0.1524" layer="91"/>
+</segment>
 </net>
 <net name="+5V" class="0">
@@
 </segment>
 </net>
+<net name="STOP" class="0">
+<segment>
+<pinref part="STOP" gate="G$1" pin="2"/>
+<wire x1="-53.34" y1="27.94" x2="-38.1" y2="27.94" width="0.1524" layer="91"/>
+<label x="-38.1" y="27.94" size="1.27" layer="95" xref="yes"/>
+</segment>
+<segment>
+<pinref part="R6" gate="G$1" pin="2"/>
+<wire x1="-20.32" y1="27.94" x2="-22.86" y2="27.94" width="0.1524" layer="91"/>
+<label x="-22.86" y="27.94" size="1.27" layer="95" rot="R180" xref="yes"/>
+</segment>
+</net>
+<net name="ADC" class="0">
+<segment>
+<pinref part="U1" gate="G$1" pin="ADC"/>
+<wire x1="35.56" y1="27.94" x2="5.08" y2="27.94" width="0.1524" layer="91"/>
+<pinref part="R5" gate="G$1" pin="2"/>
+<wire x1="5.08" y1="27.94" x2="-7.62" y2="27.94" width="0.1524" layer="91"/>
+<junction x="5.08" y="27.94"/>
+<pinref part="R6" gate="G$1" pin="1"/>
+<wire x1="-7.62" y1="27.94" x2="-10.16" y2="27.94" width="0.1524" layer="91"/>
+<wire x1="-7.62" y1="25.4" x2="-7.62" y2="27.94" width="0.1524" layer="91"/>
+<junction x="-7.62" y="27.94"/>
+<pinref part="D2" gate="G$1" pin="A"/>
+</segment>
+</net>

Commit message: Schematic annotation
Connections:
- net ADC: no longer D2.A
- net GND: now also D2.A; no longer D2.C
- net STOP: now also D2.C
Other:
- note added: "BOOTLOADER MODES"
- note added: "GPIO 0 GPIO 2 GPIO 15 0 1 0 1 1 0 0 0 1"
- note added: "GPIO0 - Green LED status indicator GPIO1 - SPI Slave Select 1 GPIO2 - Audible alarm control GPIO3 - SPI Slave Select 2 GPIO4 - RFID-DATA1 (data in) GPIO5 - RFID-DATA0 (data in) GPIO12 - SPI MOSI GPIO13 - SPI MISO GPIO14 - SPI CLK GPIO15 - APD Enable ADC - Stop / Logout"
- note added: "PIN ASSIGNMENTS"
- note added: "Stop / Logout Button"
- note added: "UART DOWNLOAD (Program) FLASH STARTUP (default) SD-Card Boot"
- note removed: "USB data lines for future peripherals"
- moved on the sheet: D2, JP3, PROG-HEADER, RFID-HEADER, SPI-HEADER, SPI_HEADER, STOP, USB

Commit message: SM v1.1
with fixes
Parts:
- removed D2: PMLL4150, diode:PMLL4150
- removed PROG-HEADER: PROG-HEADER, pinhead+:PINHD-1X6
- removed SPI_HEADER: SPI-HEADER, pinhead+:PINHD-1X5
- added D1: MMBZ5V6ALT1G, diode:BAS40-06
- added JP1: (no value), pinhead+:PINHD-1X3
- added JP4: (no value), pinhead+:PINHD-1X7
- added TP1, TP2, TP3, TP4, TP5, TP6, TP7: TPB1,27, testpad:TPB1,27
- S1: value DTSM-3 -> RESET
- S2: value DTSM-3 -> BOOT-LOADER
- SPI-HEADER: value SPI_HEADER -> (none); device pinhead+:PINHD-1X5 -> pinhead+:PINHD-1X7
- USB: value USB-HEADER -> 5V-Power
Connections:
- removed net D+: USB.2
- removed net D-: USB.3
- new net N$1: U$2G$4.P$2
- new net N$10: TP2.TP, U1.MISO
- new net N$11: TP3.TP, U1.*GPIO9
- new net N$12: TP4.TP, U1.*GPIO10
- new net N$13: TP5.TP, U1.MOSI
- new net N$15: TP6.TP, U1.SCLK
- new net N$2: U$2G$5.P$2
- new net N$3: U$2G$6.P$2
- new net N$4: U$1G$3.P$2
- new net N$5: U$1G$4.P$2
- new net N$6: U$1G$5.P$2
- new net N$7: U$1G$6.P$2
- new net N$8: TP7.TP, U1.GPIO16
- new net N$9: TP1.TP, U1.CS0
- net +3V3: now also D1.K2, JP4.7, SPI-HEADER.1; no longer PROG-HEADER.2
- net +5V: now also RFID-HEADER.6, USB.2; no longer RFID-HEADER.1
- net APD_EN: now also U$2G$3.P$2; no longer U$2G$1.P$2
- net BUZZER: now also RFID-HEADER.5, U$2G$2.P$2; no longer RFID-HEADER.4, U$2G$3.P$2
- net GND: now also D1.AA, JP1.3, JP4.1, RFID-HEADER.1, SPI-HEADER.7, USB.3; no longer D2.A, PROG-HEADER.6, RFID-HEADER.6
- net GPIO0: now also U$2G$1.P$1; no longer PROG-HEADER.1, U$2G$2.P$1
- net GPIO1: now also JP1.1, JP4.3, SPI-HEADER.5; no longer PROG-HEADER.3, SPI-HEADER.4, SPI_HEADER.4
- net GPIO12: now also JP4.5, SPI-HEADER.3; no longer SPI-HEADER.2, SPI_HEADER.2
- net GPIO13: now also JP4.4, SPI-HEADER.4; no longer SPI-HEADER.3, SPI_HEADER.3
- net GPIO14: now also JP4.6, SPI-HEADER.2; no longer SPI-HEADER.1, SPI_HEADER.1
- net GPIO15: now also U$2G$3.P$1; no longer U$2G$1.P$1
- net GPIO2: now also U$2G$2.P$1; no longer U$2G$3.P$1
- net GPIO3: now also JP1.2, JP4.2, SPI-HEADER.6; no longer PROG-HEADER.5, SPI-HEADER.5, SPI_HEADER.5
- net GPIO4: now also U$1G$2.P$2; no longer U$1G$1.P$2
- net GPIO5: now also U$1G$1.P$2; no longer U$1G$2.P$2
- net GREEN_LED: now also RFID-HEADER.4, U$2G$1.P$2; no longer RFID-HEADER.5, U$2G$2.P$2
- net RESET: no longer PROG-HEADER.4
- net RFID-DATA0: now also U$1G$1.P$1; no longer U$1G$2.P$1
- net RFID-DATA1: now also U$1G$2.P$1; no longer U$1G$1.P$1
- net STOP: now also D1.K1; no longer D2.C
Other:
- note added: "Any N.O. momentary pushbutton"
- note added: "Device power - 5V 1A"
- note added: "ESP8266 Serial & Programming Header (FTDI / Prolific)"
- note added: "For future expansion and features, display, keyboard output.. etc.. currently unused."
- note added: "Interface for HID-PROX 125kHz readers (HID Proxpro II, HID Proxpoint plus.. etc) (Wiegand protocol)"
- note added: "RX"
- note added: "TX"
- note added: "To an isolated dc-actuated power cord (NO) for controlling power to 120vac appliances. (PowerSwitch Tail II or similar)"
- note removed: "5-16V"
- note removed: "Device power and USB HID"
- note removed: "ESP8266 Serial & Programming Header"
- note removed: "NC"
- note removed: "NO CONNECT"
- moved on the sheet: C1, C2, C3, C4, C5, H1, H2, H3, H4, IC1, JP3, R1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
