File: SM/StationModule.sch (EAGLE design)
At the start: 36 parts, among them IC1 REG1117

Commit message: Issues fixed
Connections:
- net GND: now also JP3.2
Changed lines of the file:
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@@
 <wire x1="33.02" y1="149.86" x2="33.02" y2="147.32" width="0.1524" layer="91"/>
 <pinref part="SUPPLY13" gate="GND" pin="GND"/>
+<pinref part="JP3" gate="A" pin="2"/>
+<wire x1="48.26" y1="152.4" x2="48.26" y2="149.86" width="0.1524" layer="91"/>
+<junction x="48.26" y="149.86"/>
 </segment>
 <segment>
